File: stlink3-flash.kicad_pcb (KiCad board)
At the start: 2 copper layers, 19 x 24.8 mm, 10 parts, among them J1 Conn_01x04, J3 Conn_01x01, J5 Conn_01x01, J6 Conn_01x01, J7 Conn_01x01, J8 Conn_01x01, J9 Conn_01x01, U1 W25Q128JVSSIQ_TR

Commit message: add gerber
Parts:
- removed J7, J8: Conn_01x01, Connector_PinHeader_1.27mm:PinHeader_1x01_P1.27mm_Vertical
- added J2: Conn_01x02, Connector_PinHeader_1.27mm:PinHeader_1x02_P1.27mm_Vertical, F.Cu at (98.4, 50.8)
- moved U1 0.64 mm to (90.8, 47.0)
- moved C1 0.63 mm to (94.0, 52.1)
- moved R1 0.63 mm to (87.6, 52.1)
Routing:
- net GND: track 2.86 -> 4.55 mm, vias 2 -> 3
- net /~FLASH_CS~: track 21.8 -> 20.7 mm
- net /SPI4_SCK: track 19.2 -> 18.4 mm, vias 0 -> 1
- net /SPI4_MOSI: track 16.6 -> 16.4 mm, vias 0 -> 1
- net +3V3: vias 0 -> 1
